Commit message: Add missing files. Open source code now support gepetto display.

File: data/double_pendulum_rigid.urdf (robot description, URDF)
Before this commit: robot pendulum, 5 links, 4 joints
Links:
- link PendulumArm: geometry visual mesh filename=/home/builder/wdc_workspace/src/jiminy/data/PendulumArm.STL
- link PendulumMass: geometry visual mesh filename=/home/builder/wdc_workspace/src/jiminy/data/PendulumMass.STL
- link SecondPendulumArm: geometry visual mesh filename=/home/builder/wdc_workspace/src/jiminy/data/SecondPendulumA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
- link SecondPendulumMass: geometry visual mesh filename=/home/builder/wdc_workspace/src/jiminy/data/SecondPendulumM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
- link world: geometry visual mesh filename=/home/builder/wdc_workspace/src/jiminy/data/world.STL
