Commit message: Add gym cartpole openAI environment and DQN learning example.

File: data/cartpole/cartpole.urdf (robot description, URDF)
Before this commit: robot physics, 3 links, 2 joints
Joints:
- joint cart_to_pole: limit lower=-1.57 upper=1.57 effort=1000.0 velocity=1000 -> lower=-10 upper=10 effort=1000.0 velocity=1000
