Commit message: Add multiple toy models with meshes. Add standalone Exo model with meshes. Rework of python bindings for more flexibility and user-friendlyness. Move flexibility dynamics into the Engine itself.

File: data/double_pendulum/double_pendulum.urdf (robot description, URDF)
Before this commit: robot pendulum, 5 links, 4 joints
Links:
- link PendulumArm: geometry visual mesh filename=/home/builder/wdc_workspace/src/jiminy/data/double_pendulum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
- link PendulumMass: geometry visual mesh filename=/home/builder/wdc_workspace/src/jiminy/data/double_pendulum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
- link SecondPendulumArm: geometry visual mesh filename=/home/builder/wdc_workspace/src/jiminy/data/double_pendulum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
- link SecondPendulumMass: geometry visual mesh filename=/home/builder/wdc_workspace/src/jiminy/data/double_pendulum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
- link world: geometry visual mesh filename=/home/builder/wdc_workspace/src/jiminy/data/double_pendulum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

File: wdc/data/atalante_with_patient/atalante_with_patient.urdf (robot description, URDF)
Before this commit: robot v5-4, 34 links, 33 joints
Links:
- link LeftFrontalHipLink: geometry collision mesh filename=/home/builder/wdc_workspace/src/jiminy/wdc/data/atalante_wi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; visual mesh filename=/home/builder/wdc_workspace/src/jiminy/wdc/data/atalante_wi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
- link LeftHenkeAnkleLink: geometry collision mesh filename=/home/builder/wdc_workspace/src/jiminy/wdc/data/atalante_wi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; visual mesh filename=/home/builder/wdc_workspace/src/jiminy/wdc/data/atalante_wi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
- link LeftSagittalAnkleLink: geometry collision mesh filename=/home/builder/wdc_workspace/src/jiminy/wdc/data/atalante_wi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; visual mesh filename=/home/builder/wdc_workspace/src/jiminy/wdc/data/atalante_wi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
- link LeftSagittalHipLink: geometry collision mesh filename=/home/builder/wdc_workspace/src/jiminy/wdc/data/atalante_wi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; visual mesh filename=/home/builder/wdc_workspace/src/jiminy/wdc/data/atalante_wi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
- link LeftSagittalKneeLink: geometry collision mesh filename=/home/builder/wdc_workspace/src/jiminy/wdc/data/atalante_wi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; visual mesh filename=/home/builder/wdc_workspace/src/jiminy/wdc/data/atalante_wi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
- link LeftToeLink: geometry collision mesh filename=/home/builder/wdc_workspace/src/jiminy/wdc/data/atalante_wi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; visual mesh filename=/home/builder/wdc_workspace/src/jiminy/wdc/data/atalante_wi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
- link LeftTransverseHipLink: geometry collision mesh filename=/home/builder/wdc_workspace/src/jiminy/wdc/data/atalante_wi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; visual mesh filename=/home/builder/wdc_workspace/src/jiminy/wdc/data/atalante_wi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
- link PelvisLink: geometry collision mesh filename=/home/builder/wdc_workspace/src/jiminy/wdc/data/atalante_wi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; visual mesh filename=/home/builder/wdc_workspace/src/jiminy/wdc/data/atalante_wi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
- link RightFrontalHipLink: geometry collision mesh filename=/home/builder/wdc_workspace/src/jiminy/wdc/data/atalante_wi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; visual mesh filename=/home/builder/wdc_workspace/src/jiminy/wdc/data/atalante_wi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
- link RightHenkeAnkleLink: geometry collision mesh filename=/home/builder/wdc_workspace/src/jiminy/wdc/data/atalante_wi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; visual mesh filename=/home/builder/wdc_workspace/src/jiminy/wdc/data/atalante_wi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
- link RightSagittalAnkleLink: geometry collision mesh filename=/home/builder/wdc_workspace/src/jiminy/wdc/data/atalante_wi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; visual mesh filename=/home/builder/wdc_workspace/src/jiminy/wdc/data/atalante_wi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
- link RightSagittalHipLink: geometry collision mesh filename=/home/builder/wdc_workspace/src/jiminy/wdc/data/atalante_wi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; visual mesh filename=/home/builder/wdc_workspace/src/jiminy/wdc/data/atalante_wi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
- link RightSagittalKneeLink: geometry collision mesh filename=/home/builder/wdc_workspace/src/jiminy/wdc/data/atalante_wi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; visual mesh filename=/home/builder/wdc_workspace/src/jiminy/wdc/data/atalante_wi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
- link RightToeLink: geometry collision mesh filename=/home/builder/wdc_workspace/src/jiminy/wdc/data/atalante_wi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; visual mesh filename=/home/builder/wdc_workspace/src/jiminy/wdc/data/atalante_wi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
- link RightTransverseHipLink: geometry collision mesh filename=/home/builder/wdc_workspace/src/jiminy/wdc/data/atalante_wi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; visual mesh filename=/home/builder/wdc_workspace/src/jiminy/wdc/data/atalante_wi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

Commit message: Various bug fixes with open AI interface. Improve gym jiminy env 'template' style.

File: data/double_pendulum/double_pendulum.urdf (robot description, URDF)
Before this commit: robot pendulum, 5 links, 4 joints
Links:
- link PendulumMass: mass 1.0 -> 3.0
Joints:
- joint PendulumJoint: axis 1 0 0 -> 0 1 0
- joint SecondPendulumJoint: axis 1 0 0 -> 0 1 0

Commit message: WIP: Draft of Acrobot learning based on SAC-HER.

File: data/double_pendulum/double_pendulum.urdf (robot description, URDF)
Before this commit: robot pendulum, 5 links, 4 joints
Links:
- link SecondPendulumMass: mass 1.0 -> 2.0
Joints:
- joint PendulumMassJoint: origin xyz=0.0 0.0 1.0 rpy=0 0 0 -> xyz=0.0 0.0 0.5 rpy=0 0 0
- joint SecondPendulumMassJoint: origin xyz=0.0 0.0 0.5 rpy=0 0 0 -> xyz=0.0 0.0 1.0 rpy=0 0 0
